File: BMS_prototype_v0.kicad_sch (KiCad schematic)
At the start: 51 parts, among them J1 Conn_01x16_Pin, J2 Conn_01x05_Pin, J3 Conn_01x06_Pin, Q1 NPN, U1 PBQ76952PFBT, U2 BQ7697202PFBR

Commit message: Revisão de conexões
Parts:
- removed U2: BQ7697202PFBR, TQFP48_PFB_TEX, symbol BQ76972:BQ7697202PFBR
- added C21, C22: 1uF, symbol Device:C
- added C23: 22nF, symbol Device:C
- added C24: 220nF, symbol Device:C
- added R20: 10M, symbol Device:R
- added R21: R, symbol Device:R
- C1, C10, C11, C12, C2, C3, C4, C5, C6, C7, C8, C9: value C -> 220nF
- C13, C20: value C -> 1uF
- C14, C17: value C -> 100pF
- C15: value C -> 0.47uF
- C16: value C -> 0.1uF
- C18: value C -> 2.2uF
- C19: value C -> 0.01uF
- R15, R17, R18: value R -> 100
- R16: value R -> 10k
- R19: value R -> 220
- Rsense: value R -> 0.001
Connections:
- net BAT+: now also D1.2 (A), J1.4 (Pin_4), R1.2; no longer C13.1, C14.1, C15.2, R15.1, U1.47 (BAT)
- net BREG: now also R20.1
- net GND: now also C1.2, C19.2, J1.16 (Pin_16), R17.1, Rsense.1, C21.1, C22.1, C23.2, R20.2, R21.2; no longer C12.2, C19.1, U1.34 (REG2)
- net REGIN: now also C23.1
- net REG_3V3: now also C21.2
- net RST_SHUT: now also C19.1; no longer C19.2
- net VC0: now also C11.1, R21.1; no longer C12.1, R12.1
- net VC1: now also C1.1, C2.2, R12.1; no longer C10.2, C11.1, R11.1
- net VC15: now also C12.1, C24.2; no longer C1.2, C2.1
- net VC16: now also C24.1; no longer C1.1
- net VC2: now also C2.1, C3.2, R11.1; no longer C10.1, C9.2, R10.1
- net VC3: now also C3.1, C4.2, R10.1; no longer C8.2, C9.1, R9.1
- net VC4: now also C4.1, C5.2, R9.1; no longer C7.2, C8.1, R8.1
- net VC5: now also C5.1, R8.1; no longer C7.1, R7.1
- net VC6: now also C7.2, R7.1; no longer C5.2, R6.1
- net VC7: now also C7.1, C8.2, R6.1; no longer C4.2, C5.1, R5.1
- net VC8: now also C8.1, C9.2, R5.1; no longer C3.2, C4.1, R4.1
- net VC9: now also C10.2, C9.1, R4.1; no longer C2.2, C3.1, J1.2 (Pin_2), J1.3 (Pin_3), J1.4 (Pin_4), J1.5 (Pin_5), J1.6 (Pin_6), J1.7 (Pin_7), R2.2, R3.1, R3.2, U1.2 (VC14), U1.3 (VC13), U1.4 (VC12), U1.5 (VC11), U1.6 (VC10)
- net 6P: now reaches J1.10 (Pin_10)
- net 6P: now also R7.2; no longer R6.2
- net 5P: now reaches J1.11 (Pin_11)
- net 5P: now also R8.2; no longer R7.2
- net 4P: now reaches J1.12 (Pin_12)
- net 4P: now also R9.2; no longer R8.2
- net 3P: now reaches J1.13 (Pin_13)
- net 3P: now also R10.2; no longer R9.2
- net 2P: now reaches J1.14 (Pin_14)
- net 2P: now also R11.2; no longer R10.2
- net 1P: now reaches J1.15 (Pin_15)
- net 1P: now also R12.2; no longer R11.2
- net 8P: now reaches J1.8 (Pin_8)
- net 8P: now also R5.2; no longer R4.2
- net 7P: now reaches J1.9 (Pin_9)
- net 7P: now also R6.2; no longer R5.2
- net FUSE: now reaches U1.38 (FUSE)
- net PDSG: now reaches U1.39 (PDSG)
- net PCHG: now reaches U1.40 (PCHG)
- net LD: now reaches U1.41 (LD)
- net PACK: now reaches U1.42 (PACK)
- net DSG : now reaches U1.43 (DSG)
- net CHG: now reaches U1.45 (CHG)
- net at D1.1 (K): now also R15.1; no longer R15.2
- removed net BAT-: J1.16 (Pin_16), R12.2, R17.1, Rsense.1
- new net: C22.2, U1.34 (REG2)
- new net 10P: J1.6 (Pin_6), R3.2
- new net 11P: J1.5 (Pin_5), R2.2
- new net 9P: J1.7 (Pin_7), R4.2
- new net BAT: C13.1, C14.1, C15.2, R15.2, U1.47 (BAT)
- new net VC10: C10.1, C12.2, R3.1, U1.2 (VC14), U1.3 (VC13), U1.4 (VC12), U1.5 (VC11), U1.6 (VC10)
- now unconnected: J1.1 (Pin_1)
- no-connect marks 5 -> 8
Other:
- note added: "Confirmar conexão de cels não usadas"
- note added: "No datasheet GND conectado a BAT- via um Net-Tie"
- moved on the sheet: C11, C13, C14, C15, C16, C17, C18, C19, D1, J1, R1, R10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

Commit message: Revisão
Other:
- note added: "0.001 ohm é o valor selecionado no datasheet. Podemos alterar para mudar o range de medições"
- note added: "pino TS2 pode ser usado como sinal WAKE também"
Changed lines of the file:
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@@
 	)
 	(junction
-		(at 151.13 128.27)
-		(diameter 0)
-		(color 0 0 0 0)
-	)
-	(junction
 		(at 152.4 38.1)
 		(diameter 0)
@@
 	(wire
 		(pts
+			(xy 153.67 133.35) (xy 205.74 133.35)
+		)
+		(stroke
+			(width 0)
+			(type default)
+		)
+	)
+	(wire
+		(pts
 			(xy 246.38 123.19) (xy 248.92 123.19)
 		)
@@
 	(wire
 		(pts
-			(xy 184.15 133.35) (xy 184.15 142.24)
-		)
-		(stroke
-			(width 0)
-			(type default)
-		)
-	)
-	(wire
-		(pts
 			(xy 246.38 100.33) (xy 248.92 100.33)
 		)
@@
 	(wire
 		(pts
+			(xy 153.67 133.35) (xy 153.67 142.24)
+		)
+		(stroke
+			(width 0)
+			(type default)
+		)
+	)
+	(wire
+		(pts
 			(xy 151.13 142.24) (xy 153.67 142.24)
 		)
@@
 	(wire
 		(pts
-			(xy 151.13 128.27) (xy 139.7 128.27)
-		)
-		(stroke
-			(width 0)
-			(type default)
-		)
-	)
-	(wire
-		(pts
 			(xy 246.38 107.95) (xy 248.92 107.95)
 		)
@@
 	(wire
 		(pts
-			(xy 151.13 128.27) (xy 205.74 128.27)
-		)
-		(stroke
-			(width 0)
-			(type default)
-		)
-	)
-	(wire
-		(pts
 			(xy 257.81 49.53) (xy 264.16 49.53)
 		)
@@
 	(wire
 		(pts
-			(xy 184.15 133.35) (xy 205.74 133.35)
-		)
-		(stroke
-			(width 0)
-			(type default)
-		)
-	)
-	(wire
-		(pts
 			(xy 81.28 153.67) (xy 81.28 138.43)
 		)
@@
 	(wire
 		(pts
-			(xy 184.15 142.24) (xy 153.67 142.24)
-		)
-		(stroke
-			(width 0)
-			(type default)
-		)
-	)
-	(wire
-		(pts
 			(xy 30.48 160.02) (xy 33.02 160.02)
 		)
@@
 	(wire
 		(pts
-			(xy 151.13 125.73) (xy 151.13 128.27)
+			(xy 139.7 128.27) (xy 205.74 128.27)
 		)
 		(stroke
@@
 	)
 	(rectangle
+		(start 245.745 149.225)
+		(end 285.115 165.735)
+		(stroke
+			(width 0)
+			(type default)
+		)
+		(fill
+			(type none)
+		)
+	)
+	(rectangle
 		(start 187.96 16.51)
 		(end 234.95 71.755)
@@
 		)
 	)
+	(text_box "OBS1: Adicionar TestPoints\nOBS2: Selecionar Footprints\n"
+		(exclude_from_sim no)
+		(at 245.745 149.225 0)
+		(size 39.37 16.51)
+		(stroke
+			(width 0)
+			(type default)
+		)
+		(fill
+			(type none)
+		)
+		(effects
+			(font
+				(size 1.27 1.27)
+			)
+			(justify left top)
+		)
+	)
 	(text_box "Fonte de alimentação para reguladores LDO internos (REG1, REG2 e REG18). Dimensionar npn para aguentar tensão máxima de bateria e corrente máxima de fornecimento do BQ769x2(~45mA). Avaliar utilização de regulador de tensão independente.\n"
 		(exclude_from_sim no)
@@
 		)
 	)
+	(text "0.001 ohm é o valor selecionado no datasheet. \nPodemos alterar para mudar o range de medições\n"
+		(exclude_from_sim no)
+		(at 148.59 192.278 0)
+		(effects
+			(font
+				(size 0.6096 0.6096)
+			)
+		)
+	)
 	(text "Confirmar conexão de cels não usadas\n"
 		(exclude_from_sim no)
@@
 		)
 	)
+	(text "pino TS2 pode ser usado como sinal WAKE também"
+		(exclude_from_sim no)
+		(at 193.04 143.764 0)
+		(effects
+			(font
+				(size 0.6096 0.6096)
+			)
+		)
+	)
 	(text "No datasheet GND conectado a BAT- via um Net-Tie\n\n"
 		(exclude_from_sim no)
@@
 		)
 	)
+	(label "SRN"
+		(at 153.67 133.35 0)
+		(fields_autoplaced yes)
+		(effects
+			(font
+				(size 1.27 1.27)
+			)
+			(justify left bottom)
+		)
+	)
 	(label "8P"
 		(at 36.83 125.73 0)
@@
 		)
 	)
+	(label "SRP"
+		(at 139.7 128.27 0)
+		(fields_autoplaced yes)
+		(effects
+			(font
+				(size 1.27 1.27)
+			)
+			(justify left bottom)
+		)
+	)
 	(global_label "VC8"
 		(shape input)
@@
 		)
 	)
-	(global_label "SRN"
-		(shape input)
-		(at 184.15 133.35 180)
-		(fields_autoplaced yes)
-		(effects
-			(font
-				(size 1.27 1.27)
-			)
-			(justify right)
-		)
-		(property "Intersheetrefs" "${INTERSHEET_REFS}"
-			(at 177.3548 133.35 0)
-			(effects
-				(font
-					(size 1.27 1.27)
-				)
-				(justify right)
-				(hide yes)
-			)
-		)
-	)
 	(global_label "CHG"
 		(shape input)
@@
 				(hide yes)
 			)
-		)
-	)
-	(global_label "SRP"
-		(shape input)
-		(at 151.13 125.73 180)
-		(fields_autoplaced yes)
-		(effects
-			(font
-				(size 1.27 1.27)
-			)
-			(justify right)
-		)
-		(property "Intersheetrefs" "${INTERSHEET_REFS}"
-			(at 144.3953 125.73 0)
-			(effects
-				(font
-					(size 1.27 1.27)
-				)
-				(justify right)
-				(hide yes)
-			)

Commit message: Inserindo footprints
Parts:
- C1, C10, C11, C12, C13, C14, C15, C16, C17, C18, C19, C2, C20, C21, C22, C23, C24, C3, C4, C5, C6, C7, C8, C9: footprint (none) -> Capacitor_SMD:C_0402_1005Metric_Pad0.74x0.62mm_HandSolder
- D1, D2: footprint (none) -> Diode_SMD:D_SOD-123
- J1: footprint (none) -> Connector_PinHeader_2.54mm:PinHeader_1x16_P2.54mm_Vertical
- J2: footprint (none) -> Connector_PinHeader_2.54mm:PinHeader_1x05_P2.54mm_Vertical
- J3: footprint (none) -> Connector_PinHeader_2.54mm:PinHeader_1x06_P2.54mm_Vertical
- Q1: footprint (none) -> Package_TO_SOT_SMD:SOT-89-3
- R1, R10, R11, R12, R13, R14, R15, R16, R17, R18, R19, R2, R20, R21, R3, R4, R5, R6, R7, R8, R9, Rsense: footprint (none) -> Resistor_SMD:R_0402_1005Metric
- S1: footprint KMR_2 -> Footprints:SMD_Button_KMR_2
- TH1, TH2: footprint (none) -> Footprints:103AT2
- U1: footprint PFB48_TEX -> Footprints:BQ76952_TEX
Changed lines of the file:
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@@
 			)
 		)
-		(property "Footprint" ""
+		(property "Footprint" "Resistor_SMD:R_0402_1005Metric"
 			(at 253.492 24.13 90)
 			(effects
@@
 			)
 		)
-		(property "Footprint" ""
+		(property "Footprint" "Connector_PinHeader_2.54mm:PinHeader_1x16_P2.54mm_Vertical"
 			(at 25.4 125.73 0)
 			(effects
@@
 			)
 		)
-		(property "Footprint" "PFB48_TEX"
+		(property "Footprint" "Footprints:BQ76952_TEX"
 			(at 205.74 85.09 0)
 			(effects
@@
 			)
 		)
-		(property "Footprint" ""
+		(property "Footprint" "Resistor_SMD:R_0402_1005Metric"
 			(at 41.91 129.032 90)
 			(effects
@@
 			)
 		)
-		(property "Footprint" ""
+		(property "Footprint" "Capacitor_SMD:C_0402_1005Metric_Pad0.74x0.62mm_HandSolder"
 			(at 93.6752 130.81 0)
 			(effects
@@
 			)
 		)
-		(property "Footprint" ""
+		(property "Footprint" "Resistor_SMD:R_0402_1005Metric"
 			(at 41.91 123.952 90)
 			(effects
@@
 			)
 		)
-		(property "Footprint" ""
+		(property "Footprint" "Resistor_SMD:R_0402_1005Metric"
 			(at 41.91 136.652 90)
 			(effects
@@
 			)
 		)
-		(property "Footprint" ""
+		(property "Footprint" "Resistor_SMD:R_0402_1005Metric"
 			(at 41.91 113.792 90)
 			(effects
@@
 			)
 		)
-		(property "Footprint" ""
+		(property "Footprint" "Capacitor_SMD:C_0402_1005Metric_Pad0.74x0.62mm_HandSolder"
 			(at 268.9352 113.03 0)
 			(effects
@@
 			)
 		)
-		(property "Footprint" ""
+		(property "Footprint" "Capacitor_SMD:C_0402_1005Metric_Pad0.74x0.62mm_HandSolder"
 			(at 93.6752 92.71 0)
 			(effects
@@
 			)
 		)
-		(property "Footprint" ""
+		(property "Footprint" "Resistor_SMD:R_0402_1005Metric"
 			(at 147.32 191.008 90)
 			(effects
@@
 			)
 		)
-		(property "Footprint" ""
+		(property "Footprint" "Resistor_SMD:R_0402_1005Metric"
 			(at 256.032 24.13 90)
 			(effects
@@
 			)
 		)
-		(property "Footprint" ""
+		(property "Footprint" "Resistor_SMD:R_0402_1005Metric"
 			(at 41.91 141.732 90)
 			(effects
@@
 			)
 		)
-		(property "Footprint" ""
+		(property "Footprint" "Capacitor_SMD:C_0402_1005Metric_Pad0.74x0.62mm_HandSolder"
 			(at 151.13 150.1648 0)
 			(effects
@@
 			)
 		)
-		(property "Footprint" ""
+		(property "Footprint" "Capacitor_SMD:C_0402_1005Metric_Pad0.74x0.62mm_HandSolder"
 			(at 151.13 141.2748 0)
 			(effects
@@
 			)
 		)
-		(property "Footprint" ""
+		(property "Footprint" "Capacitor_SMD:C_0402_1005Metric_Pad0.74x0.62mm_HandSolder"
 			(at 93.6752 107.95 0)
 			(effects
@@
 			)
 		)
-		(property "Footprint" ""
+		(property "Footprint" "Capacitor_SMD:C_0402_1005Metric_Pad0.74x0.62mm_HandSolder"
 			(at 260.35 121.6152 0)
 			(effects
@@
 			)
 		)
-		(property "Footprint" ""
+		(property "Footprint" "Resistor_SMD:R_0402_1005Metric"
 			(at 41.91 134.112 90)
 			(effects
@@
 			)
 		)
-		(property "Footprint" ""
+		(property "Footprint" "Resistor_SMD:R_0402_1005Metric"
 			(at 41.91 121.412 90)
 			(effects
@@
 			)
 		)
-		(property "Footprint" ""
+		(property "Footprint" "Resistor_SMD:R_0402_1005Metric"
 			(at 41.91 144.272 90)
 			(effects
@@
 			)
 		)
-		(property "Footprint" ""
+		(property "Footprint" "Capacitor_SMD:C_0402_1005Metric_Pad0.74x0.62mm_HandSolder"
 			(at 93.6752 115.57 0)
 			(effects
@@
 			)
 		)
-		(property "Footprint" ""
+		(property "Footprint" "Resistor_SMD:R_0402_1005Metric"
 			(at 85.09 55.118 90)
 			(effects
@@
 			)
 		)
-		(property "Footprint" ""
+		(property "Footprint" "Resistor_SMD:R_0402_1005Metric"
 			(at 41.91 126.492 90)
 			(effects
@@
 			)
 		)
-		(property "Footprint" ""
+		(property "Footprint" "Resistor_SMD:R_0402_1005Metric"
 			(at 141.478 177.8 90)
 			(effects
@@
 			)
 		)
-		(property "Footprint" ""
+		(property "Footprint" "Resistor_SMD:R_0402_1005Metric"
 			(at 198.882 48.26 90)
 			(effects
@@
 			)
 		)
-		(property "Footprint" ""
+		(property "Footprint" "Capacitor_SMD:C_0402_1005Metric_Pad0.74x0.62mm_HandSolder"
 			(at 102.5652 50.8 0)
 			(effects
@@
 			)
 		)
-		(property "Footprint" ""
+		(property "Footprint" "Capacitor_SMD:C_0402_1005Metric_Pad0.74x0.62mm_HandSolder"
 			(at 93.6752 138.43 0)
 			(effects
@@
 			)
 		)
-		(property "Footprint" ""
+		(property "Footprint" "Capacitor_SMD:C_0402_1005Metric_Pad0.74x0.62mm_HandSolder"
 			(at 111.4552 60.96 0)
 			(effects
@@
 			)
 		)
-		(property "Footprint" ""
+		(property "Footprint" "Diode_SMD:D_SOD-123"
 			(at 76.2 53.34 0)
 			(effects
@@
 			)
 		)
-		(property "Footprint" ""
+		(property "Footprint" "Capacitor_SMD:C_0402_1005Metric_Pad0.74x0.62mm_HandSolder"
 			(at 260.35 115.2652 0)
 			(effects
@@
 			)
 		)
-		(property "Footprint" ""
+		(property "Footprint" "Capacitor_SMD:C_0402_1005Metric_Pad0.74x0.62mm_HandSolder"
 			(at 159.7152 52.07 0)
 			(effects
@@
 			)
 		)
-		(property "Footprint" ""
+		(property "Footprint" "Diode_SMD:D_SOD-123"
 			(at 215.9 30.48 0)
 			(effects
@@
 			)
 		)
-		(property "Footprint" ""
+		(property "Footprint" "Resistor_SMD:R_0402_1005Metric"
 			(at 41.91 139.192 90)
 			(effects
@@
 			)
 		)
-		(property "Footprint" ""
+		(property "Footprint" "Resistor_SMD:R_0402_1005Metric"
 			(at 41.91 131.572 90)
 			(effects
@@
 			)
 		)
-		(property "Footprint" ""
+		(property "Footprint" "Capacitor_SMD:C_0402_1005Metric_Pad0.74x0.62mm_HandSolder"
 			(at 93.6752 100.33 0)
 			(effects
@@
 			)
 		)
-		(property "Footprint" ""
+		(property "Footprint" "Resistor_SMD:R_0402_1005Metric"
 			(at 155.448 177.8 90)
 			(effects
@@
 			)
 		)
-		(property "Footprint" ""
+		(property "Footprint" "Capacitor_SMD:C_0402_1005Metric_Pad0.74x0.62mm_HandSolder"
 			(at 93.6752 123.19 0)
 			(effects
@@
 			)
 		)
-		(property "Footprint" ""
+		(property "Footprint" "Resistor_SMD:R_0402_1005Metric"
 			(at 41.91 118.872 90)
 			(effects
@@
 			)
 		)
-		(property "Footprint" ""
+		(property "Footprint" "Capacitor_SMD:C_0402_1005Metric_Pad0.74x0.62mm_HandSolder"
 			(at 204.7748 143.51 0)
 			(effects
@@
 			)
 		)
-		(property "Footprint" ""
+		(property "Footprint" "Connector_PinHeader_2.54mm:PinHeader_1x05_P2.54mm_Vertical"
 			(at 269.24 31.75 0)
 			(effects
@@
 			)
 		)
-		(property "Footprint" ""
+		(property "Footprint" "Package_TO_SOT_SMD:SOT-89-3"
 			(at 276.86 52.07 0)
 			(effects
@@
 			)
 		)
-		(property "Footprint" ""
+		(property "Footprint" "Capacitor_SMD:C_0402_1005Metric_Pad0.74x0.62mm_HandSolder"
 			(at 93.6752 161.29 0)
 			(effects
@@
 			)
 		)
-		(property "Footprint" ""
+		(property "Footprint" "Resistor_SMD:R_0402_1005Metric"
 			(at 214.122 38.1 90)
 			(effects
@@
 			)
 		)
-		(property "Footprint" ""
+		(property "Footprint" "Capacitor_SMD:C_0402_1005Metric_Pad0.74x0.62mm_HandSolder"
 			(at 65.7352 177.8 0)
 			(effects
@@
 			)
 		)
-		(property "Footprint" ""
+		(property "Footprint" "Footprints:103AT2"
 			(at 191.77 151.13 0)
 			(effects
@@
 			)
 		)
-		(property "Footprint" ""
+		(property "Footprint" "Capacitor_SMD:C_0402_1005Metric_Pad0.74x0.62mm_HandSolder"
 			(at 78.4352 175.26 0)
 			(effects
@@
 			)
 		)
-		(property "Footprint" ""
+		(property "Footprint" "Connector_PinHeader_2.54mm:PinHeader_1x06_P2.54mm_Vertical"
 			(at 269.24 52.07 0)
 			(effects
@@
 			)
 		)
-		(property "Footprint" ""
+		(property "Footprint" "Footprints:103AT2"
 			(at 198.12 151.13 0)
 			(effects
@@
 			)
 		)
-		(property "Footprint" "KMR_2"
+		(property "Footprint" "Footprints:SMD_Button_KMR_2"
 			(at 168.91 130.48 0)
 			(effects
@@
 			)
 		)
-		(property "Footprint" ""
+		(property "Footprint" "Capacitor_SMD:C_0402_1005Metric_Pad0.74x0.62mm_HandSolder"
 			(at 224.79 43.4848 0)
 			(effects
@@
 			)
 		)
-		(property "Footprint" ""
+		(property "Footprint" "Resistor_SMD:R_0402_1005Metric"
 			(at 41.91 116.332 90)
 			(effects
@@
 			)
 		)
-		(property "Footprint" ""
+		(property "Footprint" "Capacitor_SMD:C_0402_1005Metric_Pad0.74x0.62mm_HandSolder"
 			(at 93.6752 146.05 0)
 			(effects
@@
 			)
 		)
-		(property "Footprint" ""
+		(property "Footprint" "Capacitor_SMD:C_0402_1005Metric_Pad0.74x0.62mm_HandSolder"
 			(at 93.6752 153.67 0)
 			(effects
@@
 			)
 		)
-		(property "Footprint" ""
+		(property "Footprint" "Capacitor_SMD:C_0402_1005Metric_Pad0.74x0.62mm_HandSolder"
 			(at 102.5652 60.96 0)
 			(effects
@@
 			)
 		)
-		(property "Footprint" ""
+		(property "Footprint" "Resistor_SMD:R_0402_1005Metric"
 			(at 150.622 48.26 90)
 			(effects
@@
 			)
 		)
-		(property "Footprint" ""
+		(property "Footprint" "Capacitor_SMD:C_0402_1005Metric_Pad0.74x0.62mm_HandSolder"
 			(at 93.6752 85.09 0)
 			(effects

Commit message: adiciona folha do esquemático de proteção
Other:
- note added: "pino TS2 pode ser usado como sinal WAKE também. Se for usado shutdown será necessário conectar um botão à esse pino"
- note removed: "pino TS2 pode ser usado como sinal WAKE também"
