File: BatteryProtection_v0.kicad_sch (KiCad schematic)
At the start: 0 parts

Commit message: adiciona folha do esquemático de proteção
Parts:
- added C25, C26, C27, C28: 0.1uF, symbol Device:C
- added D3, D5: 16V, symbol Device:D
- added D4: 100V, symbol Device:D
- added F1: ITV4030L1412NR, ITV4030L1412NR, symbol ITV4030L1412NR:ITV4030L1412NR
- added Q2, Q3: Q_NMOS_GSD, symbol Device:Q_NMOS_GSD
- added R22, R26: 10M, symbol Device:R
- added R23, R24, R25, R28, R29, R30, R31: 5.1k, symbol Device:R
- added R27: 7.5k, symbol Device:R
Connections:
- new net: D5.1 (K), Q3.1 (G), R24.1, R26.2, R27.1
- new net: R24.2, R25.1
- new net: C25.2, C26.1
- new net: C27.1, C28.2
- new net: R28.2, R29.1
- new net: D3.1 (K), Q2.1 (G), R22.2, R23.1
- new net: R30.2, R31.1
- new net: D4.2 (A), R27.2
- new net BAT+: C25.1, D3.2 (A), Q2.2 (S), R22.1
- new net CD: Q2.3 (D), Q3.3 (D)
- new net CHG: R23.2
- new net DSG : D4.1 (K), R25.2
- new net LD: R29.2
- new net PACK: R31.2
- new net PACK-: C26.2, C27.2, C28.1, D5.2 (A), Q3.2 (S), R26.1, R28.1, R30.1
Other:
- note added: "Fusível controlável"
