File: BMS_prototype_v0.kicad_pcb (KiCad board)
At the start: 2 copper layers, 124.8 x 94.7 mm, 134 parts, among them J1 Conn_02x12_Odd_Even, J2 Conn_01x13_Pin, J3 Conn_01x02_Pin, J4 Conn_01x02_Pin, J5 Conn_02x08_Odd_Even, J7 Conn_01x03_Pin, Q2 Q_NMOS_GSD, Q3 Q_NMOS_GSD, Q4 Q_NMOS_GSD, Q5 Q_NMOS_GSD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

Commit message: Ajustes no layout do BMS
Routing:
- net REG1_3V3: track 128.3 -> 155.1 mm, vias 2 -> 5
- net RST_SHUT: track 135.4 -> 147.7 mm, vias 0 -> 2
- net CD: track 65.4 -> 62.1 mm
- net REG2: track 72.0 -> 70.8 mm
- net EXTTS2: track 37.8 -> 38.5 mm
- net FUSE: track 16.2 -> 16.8 mm
- net GND: track 124.2 -> 124.7 mm
